Commit message: Small fixes to make work with course layout

File: ros_ws/src/bluerov2/bluerov2_description/robots/altimeter_sss.xacro (robot description, xacro)
@@ -28,4 +28,7 @@
     </gazebo>
   </xacro:bluerov2_base>
+  <xacro:bluerov_camera namespace="$(arg namespace)" parent_link="$(arg namespace)/base_link" suffix="_front">
+    <origin xyz="0.25 0.0 0.0" rpy="0 0 0"/>
+  </xacro:bluerov_camera>
   <xacro:bluerov_altimeter namespace="$(arg namespace)" parent_link="$(arg namespace)/base_link" suffix="_down">
     <origin xyz="0.05 -0.07 -0.17" rpy="0 ${0.5*pi} 0"/>

File: ros_ws/src/uuv_simulator/uuv_sensor_plugins/uuv_sensor_ros_plugins/urdf/camera_snippets.xacro (robot description, xacro)
@@ -123,5 +123,5 @@
         <plugin name="camera${suffix}_controller" filename="libgazebo_ros_camera.so">
           <updateRate>${update_rate}</updateRate>
-          <cameraName>${namespace}/camera${suffix}</cameraName>
+          <cameraName>camera${suffix}</cameraName>
           <frameName>camera${suffix}_link_optical</frameName>
           <attenuationR>0.0</attenuationR>
