Commit message: add training session 6

File: ros_ws/src/uuv_simulator/uuv_sensor_plugins/uuv_sensor_ros_plugins/urdf/imu_snippets.xacro (robot description, xacro)
@@ -22,6 +22,5 @@
     </collision>
   </xacro:macro>
-  <xacro:macro name="default_imu" params="namespace parent_link *origin">
-    <!-- ADIS16448 IMU. -->
+  <!--xacro:macro name="default_imu" params="namespace parent_link *origin">
     <xacro:imu_plugin_macro
       namespace="${namespace}"
@@ -39,4 +38,28 @@
       accelerometer_turn_on_bias_sigma="0.1960"
       orientation_noise="0.01"
+      enable_local_ned_frame="false"
+      reference_frame="world"
+      update_rate="50">
+      <inertia ixx="0.00001" ixy="0.0" ixz="0.0" iyy="0.00001" iyz="0.0" izz="0.00001" />
+      <xacro:insert_block name="origin" />
+    </xacro:imu_plugin_macro>
+  </xacro:macro-->
+  <xacro:macro name="default_imu" params="namespace parent_link *origin">
+    <!-- ADIS16448 IMU. -->
+    <xacro:imu_plugin_macro
+      namespace="${namespace}"
+      imu_suffix=""
+      parent_link="${parent_link}"
+      imu_topic="imu"
+      mass_imu_sensor="0.015"
+      gyroscope_noise_density="0.003394"
+      gyroscope_random_walk="0.00038785"
+      gyroscope_bias_correlation_time="1000.0"
+      gyroscope_turn_on_bias_sigma="0.087"
+      accelerometer_noise_density="0.04"
+      accelerometer_random_walk="0.06"
+      accelerometer_bias_correlation_time="300.0"
+      accelerometer_turn_on_bias_sigma="0.1960"
+      orientation_noise="0.03"
       enable_local_ned_frame="false"
       reference_frame="world"
